File: sweep-squared.kicad_pcb (KiCad board)
At the start: 2 copper layers, 236.3 x 106.6 mm, 76 parts, among them U1 ProMicro

Commit message: Rev 0.2
Removed questionable back silkscreen
Fixed thumb keys position (barely visible)
Fixed bat. switch position
Fixed many labels
Fixed logo
Added 5 holes for case potential
Parts:
- removed the G*** at (153.7, 88.9)
- added REF**: MountingHole_2.2mm_M2, MountingHole:MountingHole_2.2mm_M2, F.Cu at (128.6, 66.0)
- added REF**: MountingHole_2.2mm_M2, MountingHole:MountingHole_2.2mm_M2, F.Cu at (244.6, 105.4)
- added REF**: MountingHole_2.2mm_M2, MountingHole:MountingHole_2.2mm_M2, F.Cu at (188.0, 66.2)
- added REF**: MountingHole_2.2mm_M2, MountingHole:MountingHole_2.2mm_M2, F.Cu at (158.6, 146.9)
- added REF**: MountingHole_2.2mm_M2, MountingHole:MountingHole_2.2mm_M2, F.Cu at (72.4, 105.5)
- Bat +: renamed from Bat+1
- Bat -: renamed from BatGND1
- moved G*** 15.0 mm to (148.4, 120.5), turned to 40 degrees
- moved BAT_PWR 3.57 mm to (180.6, 62.6)
- moved D32 0.99 mm to (134.5, 136.0)
- moved D33 0.98 mm to (182.3, 136.1)
- moved MX31 0.38 mm to (120.0, 133.3)
- moved MX32 0.36 mm to (136.1, 146.0)
- moved D31 0.36 mm to (115.1, 124.4)
- renumbered SW_POWER1 to BAT_PWR
Routing:
- net col5: track 69.6 -> 100.5 mm
- net col1: track 214.9 -> 242.9 mm
- net row4: track 239.5 -> 260.4 mm
- net row3: track 522.8 -> 543.0 mm
- net col3: track 299.7 -> 319.3 mm
- net col2: track 207.5 -> 224.0 mm
- net Net-(D14-Pad2): track 22.6 -> 8.61 mm
- net Net-(D4-Pad2): track 21.9 -> 8.62 mm
- net col4: track 262.9 -> 275.8 mm
- net Net-(D5-Pad2): track 21.7 -> 9.55 mm
- net gnd: track 37.1 -> 46.9 mm
- net Net-(D33-Pad2): track 33.7 -> 27.6 mm
- net Net-(D7-Pad2): track 12.0 -> 17.5 mm
- net BT+: track 20.0 -> 16.1 mm
- net raw: track 35.8 -> 32.2 mm
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Other:
- board text added: "Face Down"
- board text added: "JLCJLCJLCJLC"
- board text added: "rev 0.2"
- board text removed: "Face Up"
